File: hephaestus-brain-pcb-SMT-MIXED-jig.sch (KiCad schematic (older format))
At the start: 34 parts, among them J1 Conn_01x19_Female, J2 Conn_01x19_Female, J3 Barrel_Jack, J4 Conn_01x11_Female, SW1 SW_Push

Commit message: finished jig pcb
Parts:
- gave numbers to parts that had none: 1
Changed lines of the file:
@@
 sw
 $Comp
-L power:GND #PWR?
+L power:GND #PWR0112
 U 1 1 5FC14090
 P 10550 2450
-F 0 "#PWR?" H 10550 2200 50  0001 C CNN
+F 0 "#PWR0112" H 10550 2200 50  0001 C CNN
 F 1 "GND" V 10555 2322 50  0000 R CNN
 F 2 "" H 10550 2450 50  0001 C CNN
@@
 	10150 2450 10050 2450
 $Comp
-L Device:R_Small R?
+L Device:R_Small R12
 U 1 1 5FC156B9
 P 10050 2350
-F 0 "R?" H 10109 2396 50  0000 L CNN
+F 0 "R12" H 10109 2396 50  0000 L CNN
 F 1 "10k" H 10109 2305 50  0000 L CNN
 F 2 "Resistor_SMD:R_0603_1608Metric" H 10050 2350 50  0001 C CNN
@@
 	10050 2450 9900 2450
 $Comp
-L power:+3V3 #PWR?
+L power:+3V3 #PWR0113
 U 1 1 5FC15F6A
 P 13050 1100
-F 0 "#PWR?" H 13050 950 50  0001 C CNN
+F 0 "#PWR0113" H 13050 950 50  0001 C CNN
 F 1 "+3V3" V 13065 1228 50  0000 L CNN
 F 2 "" H 13050 1100 50  0001 C CNN
@@
 $EndComp
 $Comp
-L power:+3V3 #PWR?
+L power:+3V3 #PWR0114
 U 1 1 5FC16DBE
 P 10050 2250
-F 0 "#PWR?" H 10050 2100 50  0001 C CNN
+F 0 "#PWR0114" H 10050 2100 50  0001 C CNN
 F 1 "+3V3" H 10065 2423 50  0000 C CNN
 F 2 "" H 10050 2250 50  0001 C CNN
