File: hephaestus-brain-pcb-SMT.sch (KiCad schematic (older format))
At the start: 32 parts, among them IC1 ATSAMD51G19A-MU, J1 Barrel_Jack, J2 Conn_02x03_Odd_Even, J3 USB_B_Micro, J4 Conn_02x10_Odd_Even, J5 Conn_01x03_Male, J6 Conn_01x03_Male, J7 Conn_01x03_Male, SW1 SW_SPDT, SW2 SW_SPST, SW3 SW_SPST, U1 LM1117-5.0, U2 AP2112K-3.3, U3 AT25xxx-MA, U4 74LVC1G125

Commit message: updated footprints
Parts:
- U3: footprint Package_DFN_QFN:DFN-8-1EP_3x2mm_P0.5mm_EP1.75x1.45mm -> unified:DFN-8-1EP_3x2mm_P0.5mm_EP1.75x1.45mm
Changed lines of the file:
@@
 F 0 "U3" H 6500 6100 50  0000 C CNN
 F 1 "AT25xxx-MA" H 7050 6100 50  0000 C CNN
-F 2 "Package_DFN_QFN:DFN-8-1EP_3x2mm_P0.5mm_EP1.75x1.45mm" H 6750 5850 50  0001 C CNN
+F 2 "unified:DFN-8-1EP_3x2mm_P0.5mm_EP1.75x1.45mm" H 6750 5850 50  0001 C CNN
 F 3 "http://ww1.microchip.com/downloads/en/DeviceDoc/Atmel-8707-SEEPROM-AT25010B-020B-040B-Datasheet.pdf" H 6750 5850 50  0001 C CNN
 	1    6750 5850
